File: 1.PCB/manhole.sch (EAGLE design)
At the start: 22 parts, among them IC1 7805TV

Commit message: Revert "updated PCB"
This reverts commit e032bd37680646525048ee8d74092bea044d5abf.
Parts:
- removed MQ1: (no value), jumper:JP4E
- added MQ03: (no value), jumper:JP4E
- added U$1: 5MMRGBLED, led_rgb:5MMRGBLED
Connections:
- removed net D0: JP2.15, NANO.D0/TX
- removed net MQ6A0: JP1.10, MQ1.2, MQ7.2, NANO.A2
- new net MQ135D0: MQ135.3
- new net MQ2D0: MQ2.3
- new net MQ3A0: JP1.11, MQ03.4, NANO.A1
- new net MQ3D0: MQ03.3
- new net MQ7D0: MQ7.3
- new net SS: JP2.3, NANO.D10
- net 5V: now also MQ03.1, MQ2.1, MQ7.1; no longer MQ135.2
- net BLUE: now also U$1.BLUE; no longer MQ2.1
- net GND: now also MQ03.2, MQ135.2, MQ2.2, MQ7.2, U$1.GND; no longer MQ135.3, MQ135.4, MQ2.3
- net GREEN: now also U$1.GREEN; no longer MQ2.2
- net MQ135A0: now also MQ135.4; no longer MQ1.4, MQ7.4
- net MQ2A0: now also JP1.10, MQ2.4, NANO.A2; no longer JP1.9, MQ1.1, MQ7.1, NANO.A3
- net MQ7A0: now also JP1.9, MQ7.4, NANO.A3; no longer JP1.11, MQ1.3, MQ7.3, NANO.A1
- net RED: now also U$1.RED; no longer MQ2.4
- net RED1: now also JP2.15, NANO.D0/TX; no longer JP2.3, NANO.D10
Other:
- moved on the sheet: MQ2
