File: 1.PCB/manhole.brd (EAGLE design)
At the start: 66.3 x 76.5 mm, 21 parts, among them IC1 7805TV

Commit message: PCB added
Routing:
- net GND: track 253.8 -> 269.6 mm
- net 5V: track 240.2 -> 244.0 mm
- net SCK: track 24.6 -> 23.2 mm
- net RST: track 42.0 -> 43.3 mm

Commit message: Add files via upload
Parts:
- added GSM, SPRAY: (no value), jumper:JP4
- DISP: device Wurth_Elektronik_Electromechanic_Wire_to_Board_Connectors_rev19a:612008235121 -> jumper:JP4
- moved NAV_BUTTON 12.4 mm to (6.43, 26.3)
- moved DISP 6.92 mm to (40.8, 10.9)
- moved R3 4.75 mm to (54.3, 67.3)
- moved R1 3.86 mm to (62.1, 66.8)
- moved R2 3.51 mm to (58.0, 66.3)
- moved U$1 2.87 mm to (59.5, 71.5)
Connections:
- removed net A0: JP1.12, NANO.19
- removed net D0: JP2.15, NANO.1
- removed net D2: JP2.11, NANO.5
- removed net D3: JP2.10, NANO.6
- removed net D4: JP2.9, NANO.7
- removed net D5: JP2.8, NANO.8
- removed net GND_1: JP2.12, NANO.4
- removed net N$3: DISP.2
- removed net N$5: DISP.6
- new net D9: JP2.4, NANO.12
- new net IN1: JP2.11, NANO.5, SPRAY.3
- new net IN2: JP2.8, NANO.8, SPRAY.4
- new net RX_GSM: GSM.3, JP2.10, NANO.6
- new net SCL: DISP.4, JP1.7, NANO.24
- new net SDA: DISP.3, JP1.8, NANO.23
- new net TX_GSM: GSM.4, JP2.9, NANO.7
- net 5V: now also GSM.1, SPRAY.1
- net BACK: no longer JP2.4, NANO.12
- net GND: now also DISP.2, GSM.2, JP2.12, NANO.4, SPRAY.2; no longer DISP.8
- net MOSI: no longer DISP.5
- net MQ135A0: now also JP1.12, NANO.19; no longer JP1.8, NANO.23
- net RED1: now also JP2.15, NANO.1; no longer JP1.7, NANO.24
- net RST: no longer DISP.4
- net SCK: no longer DISP.7
- net SS: no longer DISP.3
Routing:
- net GND: track 269.6 -> 318.4 mm
- net IN1: track 0.00 -> 48.7 mm
- net IN2: track 0.00 -> 41.9 mm
- net SCL: track 0.00 -> 37.8 mm
- net RST: track 43.3 -> 6.89 mm, vias 2 -> 0
- net SDA: track 0.00 -> 33.3 mm
- net BACK: track 30.2 -> 0.00 mm, vias 2 -> 0
- net SS: track 24.4 -> 6.35 mm
- net RX_GSM: track 0.00 -> 17.8 mm
- net TX_GSM: track 0.00 -> 17.6 mm
- net SCK: track 23.2 -> 6.39 mm, vias 2 -> 0
- net MOSI: track 20.8 -> 6.35 mm
- net RED1: track 36.9 -> 49.4 mm, vias 0 -> 2
- net MQ135A0: track 21.9 -> 33.6 mm, vias 0 -> 1
- net GND_1: track 6.35 -> 0.00 mm
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Other:
- board text removed: "MANHOLE"

Commit message: updated PCB
Parts:
- removed MQ03: (no value), jumper:JP4
- removed U$1: 5MMRGBLED, led_rgb:LED5MMRGB
- added MQ1: (no value), jumper:JP4
- moved MQ2 47.4 mm to (52.8, 68.6), turned to 90 degrees
- moved R1 14.9 mm to (48.2, 72.1), turned to 0 degrees
- moved MQ7 7.66 mm to (54.7, 29.3)
- moved MQ135 7.48 mm to (59.7, 40.8), turned to 180 degrees
- moved R3 4.89 mm to (58.1, 64.2), turned to 180 degrees
- moved R2 1.74 mm to (59.2, 67.6), turned to 180 degrees
Connections:
- removed net MQ135D0: MQ135.3
- removed net MQ2D0: MQ2.3
- removed net MQ3A0: JP1.11, MQ03.4, NANO.20
- removed net MQ3D0: MQ03.3
- removed net MQ7D0: MQ7.3
- removed net SS: JP2.3, NANO.13
- new net D0: JP2.15, NANO.1
- new net MQ6A0: JP1.10, MQ1.2, MQ7.2, NANO.21
- net 5V: now also MQ135.2; no longer MQ03.1, MQ2.1, MQ7.1
- net BLUE: now also MQ2.1; no longer U$1.P$1
- net GND: now also MQ135.3, MQ135.4, MQ2.3; no longer MQ03.2, MQ135.2, MQ2.2, MQ7.2, U$1.P$3
- net GREEN: now also MQ2.2; no longer U$1.P$2
- net MQ135A0: now also MQ1.4, MQ7.4; no longer MQ135.4
- net MQ2A0: now also JP1.9, MQ1.1, MQ7.1, NANO.22; no longer JP1.10, MQ2.4, NANO.21
- net MQ7A0: now also JP1.11, MQ1.3, MQ7.3, NANO.20; no longer JP1.9, MQ7.4, NANO.22
- net RED: now also MQ2.4; no longer U$1.P$4
- net RED1: now also JP2.3, NANO.13; no longer JP2.15, NANO.1
Routing:
- net GND: track 318.4 -> 253.6 mm
- net 5V: track 244.6 -> 202.0 mm
- net MQ3A0: track 37.8 -> 0.00 mm
- net RED1: track 49.4 -> 15.0 mm, vias 2 -> 1
- net MQ6A0: track 0.00 -> 17.2 mm
- net MQ135A0: track 33.6 -> 17.2 mm, vias 1 -> 0
- net MQ2A0: track 29.3 -> 17.2 mm
- net GREEN1: track 36.1 -> 47.4 mm
- net SS: track 6.35 -> 0.00 mm
- net D0: track 0.00 -> 6.35 mm
- net MQ7A0: track 19.0 -> 17.2 mm
- net GREEN: track 3.85 -> 5.54 mm
- net BLUE1: track 32.8 -> 34.2 mm
- net BLUE: track 5.32 -> 4.63 mm

Commit message: Revert "updated PCB"
This reverts commit e032bd37680646525048ee8d74092bea044d5abf.
Parts:
- removed MQ1: (no value), jumper:JP4
- added MQ03: (no value), jumper:JP4
- added U$1: 5MMRGBLED, led_rgb:LED5MMRGB
- moved MQ2 47.4 mm to (59.6, 21.6), turned to 270 degrees
- moved R1 14.9 mm to (62.1, 66.8), turned to 270 degrees
- moved MQ7 7.66 mm to (60.1, 34.8)
- moved MQ135 7.48 mm to (60.1, 48.3), turned to 270 degrees
- moved R3 4.89 mm to (54.3, 67.3), turned to 270 degrees
- moved R2 1.74 mm to (58.0, 66.3), turned to 270 degrees
Connections:
- removed net D0: JP2.15, NANO.1
- removed net MQ6A0: JP1.10, MQ1.2, MQ7.2, NANO.21
- new net MQ135D0: MQ135.3
- new net MQ2D0: MQ2.3
- new net MQ3A0: JP1.11, MQ03.4, NANO.20
- new net MQ3D0: MQ03.3
- new net MQ7D0: MQ7.3
- new net SS: JP2.3, NANO.13
- net 5V: now also MQ03.1, MQ2.1, MQ7.1; no longer MQ135.2
- net BLUE: now also U$1.P$1; no longer MQ2.1
- net GND: now also MQ03.2, MQ135.2, MQ2.2, MQ7.2, U$1.P$3; no longer MQ135.3, MQ135.4, MQ2.3
- net GREEN: now also U$1.P$2; no longer MQ2.2
- net MQ135A0: now also MQ135.4; no longer MQ1.4, MQ7.4
- net MQ2A0: now also JP1.10, MQ2.4, NANO.21; no longer JP1.9, MQ1.1, MQ7.1, NANO.22
- net MQ7A0: now also JP1.9, MQ7.4, NANO.22; no longer JP1.11, MQ1.3, MQ7.3, NANO.20
- net RED: now also U$1.P$4; no longer MQ2.4
- net RED1: now also JP2.15, NANO.1; no longer JP2.3, NANO.13
Routing:
- net GND: track 253.6 -> 318.4 mm
- net 5V: track 202.0 -> 244.6 mm
- net MQ3A0: track 0.00 -> 37.8 mm
- net RED1: track 15.0 -> 49.4 mm, vias 1 -> 2
- net MQ6A0: track 17.2 -> 0.00 mm
- net MQ135A0: track 17.2 -> 33.6 mm, vias 0 -> 1
- net MQ2A0: track 17.2 -> 29.3 mm
- net GREEN1: track 47.4 -> 36.1 mm
- net SS: track 0.00 -> 6.35 mm
- net D0: track 6.35 -> 0.00 mm
- net MQ7A0: track 17.2 -> 19.0 mm
- net GREEN: track 5.54 -> 3.85 mm
- net BLUE1: track 34.2 -> 32.8 mm
- net BLUE: track 4.63 -> 5.32 mm
